Commit message: Phase 4 complete: Gazebo simulation and robot spawning

File: ros2_ws/src/my_assembly_description/urdf/my_assembly.xacro (robot description, xacro)
@@ -314,75 +314,123 @@
   <child link="Lidar_mount_1"/>
 </joint>
-<joint name="upper_leg_fl_joint" type="continuous">
+<joint name="upper_leg_fl_joint" type="revolute">
   <origin xyz="-0.0725 -0.075 0.03" rpy="0 0 0"/>
   <parent link="base_link"/>
   <child link="Upper_leg_1"/>
   <axis xyz="0.0 -1.0 0.0"/>
-</joint>
-<joint name="upper_leg_fr_joint" type="continuous">
+  <limit lower="-1.57"
+       upper="1.57"
+       effort="50"
+       velocity="10"/>
+</joint>
+<joint name="upper_leg_fr_joint" type="revolute">
   <origin xyz="-0.0725 0.075 0.03" rpy="0 0 0"/>
   <parent link="base_link"/>
   <child link="Upper_leg_2"/>
   <axis xyz="0.0 1.0 0.0"/>
-</joint>
-<joint name="upper_leg_rl_joint" type="continuous">
+  <limit lower="-1.57"
+       upper="1.57"
+       effort="50"
+       velocity="10"/>
+</joint>
+<joint name="upper_leg_rl_joint" type="revolute">
   <origin xyz="0.0725 -0.075 0.03" rpy="0 0 0"/>
   <parent link="base_link"/>
   <child link="Upper_leg_3"/>
   <axis xyz="0.0 -1.0 0.0"/>
-</joint>
-<joint name="upper_leg_rr_joint" type="continuous">
+  <limit lower="-1.57"
+       upper="1.57"
+       effort="50"
+       velocity="10"/>
+</joint>
+<joint name="upper_leg_rr_joint" type="revolute">
   <origin xyz="0.0725 0.075 0.03" rpy="0 0 0"/>
   <parent link="base_link"/>
   <child link="Upper_leg_4"/>
   <axis xyz="0.0 1.0 0.0"/>
-</joint>
-<joint name="lower_leg_fl_joint" type="continuous">
+  <limit lower="-1.57"
+       upper="1.57"
+       effort="50"
+       velocity="10"/>
+</joint>
+<joint name="lower_leg_fl_joint" type="revolute">
   <origin xyz="0.0 0.0 -0.09" rpy="0 0 0"/>
   <parent link="Upper_leg_1"/>
   <child link="Lower_leg_1"/>
   <axis xyz="0.0 1.0 0.0"/>
-</joint>
-<joint name="lower_leg_fr_joint" type="continuous">
+  <limit lower="-2.2"
+       upper="0.3"
+       effort="50"
+       velocity="10"/>
+</joint>
+<joint name="lower_leg_fr_joint" type="revolute">
   <origin xyz="0.0 0.0 -0.09" rpy="0 0 0"/>
   <parent link="Upper_leg_2"/>
   <child link="Lower_leg_2"/>
   <axis xyz="0.0 -1.0 0.0"/>
-</joint>
-<joint name="lower_leg_rl_joint" type="continuous">
+  <limit lower="-2.2"
+       upper="0.3"
+       effort="50"
+       velocity="10"/>
+</joint>
+<joint name="lower_leg_rl_joint" type="revolute">
   <origin xyz="0.0 0.0 -0.09" rpy="0 0 0"/>
   <parent link="Upper_leg_3"/>
   <child link="Lower_leg_3"/>
   <axis xyz="-0.0 1.0 0.0"/>
-</joint>
-<joint name="lower_leg_rr_joint" type="continuous">
+  <limit lower="-2.2"
+       upper="0.3"
+       effort="50"
+       velocity="10"/>
+</joint>
+<joint name="lower_leg_rr_joint" type="revolute">
   <origin xyz="0.0 0.0 -0.09" rpy="0 0 0"/>
   <parent link="Upper_leg_4"/>
   <child link="Lower_leg_4"/>
   <axis xyz="0.0 1.0 0.0"/>
-</joint>
-<joint name="foot_fl_joint" type="continuous">
+  <limit lower="-2.2"
+       upper="0.3"
+       effort="50"
+       velocity="10"/>
+</joint>
+<joint name="foot_fl_joint" type="revolute">
   <origin xyz="-0.056132 0.0 -0.051131" rpy="0 0 0"/>
   <parent link="Lower_leg_1"/>
   <child link="Foot_1"/>
   <axis xyz="-0.0 -1.0 -0.0"/>
-</joint>
-<joint name="foot_fr_joint" type="continuous">
+  <limit lower="-1.5"
+       upper="1.5"
+       effort="30"
+       velocity="10"/>
+</joint>
+<joint name="foot_fr_joint" type="revolute">
   <origin xyz="-0.056132 0.0 -0.051131" rpy="0 0 0"/>
   <parent link="Lower_leg_2"/>
   <child link="Foot_2"/>
   <axis xyz="0.0 -1.0 0.0"/>
-</joint>
-<joint name="foot_rl_joint" type="continuous">
+  <limit lower="-1.5"
+       upper="1.5"
+       effort="30"
+       velocity="10"/>
+</joint>
+<joint name="foot_rl_joint" type="revolute">
   <origin xyz="-0.056132 0.0 -0.051131" rpy="0 0 0"/>
   <parent link="Lower_leg_3"/>
   <child link="Foot_3"/>
   <axis xyz="0.0 -1.0 -0.0"/>
-</joint>
-<joint name="foot_rr_joint" type="continuous">
+  <limit lower="-1.5"
+       upper="1.5"
+       effort="30"
+       velocity="10"/>
+</joint>
+<joint name="foot_rr_joint" type="revolute">
   <origin xyz="-0.056132 0.0 -0.051131" rpy="0 0 0"/>
   <parent link="Lower_leg_4"/>
   <child link="Foot_6"/>
   <axis xyz="0.0 -1.0 -0.0"/>
+  <limit lower="-1.5"
+       upper="1.5"
+       effort="30"
+       velocity="10"/>
 </joint>
 </robot>
